File: PCB Design/SCH_Speed-Limit-Display_2026-03-29_v45_2026-04-01-11-26/Speed-Limit-Display-v2/Speed-Limit-Display-v2.kicad_sch (KiCad schematic)
At the start: 26 parts, among them J1 USB_C_Receptacle, J2 Conn_01x12_Pin, J3 Conn_Coaxial, SW1 RotaryEncoder_Switch, SW3 SW_Push, SW4 SW_Push, U1 ESP32-S3-WROOM-1, U2 L70-R, U3 TLV75530PDBV, U4 USBLC6-2P6

Commit message: feat: complete PCB layout with full routing, GND pour, and DRC passing
PCB layout fully routed in KiCad with all traces connected, GND copper
pour on both layers, stitching vias, and custom DRC rules for USB-C
connector clearance. Updated PCB design docs and DRC checklist to
reflect current state. Board is ready for Gerber generation.

Co-Authored-By: Claude Opus 4.6 (1M context) <noreply@anthropic.com>
Parts:
- added R7, R8: 22, Resistor_SMD:R_0603_1608Metric, symbol Device:R
- BZ1: footprint (none) -> Buzzer_Beeper:Buzzer_Murata_PKMCS0909E
- C1, C3, C4, C5: footprint (none) -> Capacitor_SMD:C_0603_1608Metric
- C2, C6: footprint (none) -> Capacitor_SMD:C_0805_2012Metric
- D1: footprint (none) -> LED_SMD:LED_0603_1608Metric
- D2: footprint (none) -> Diode_SMD:D_SOD-323
- F1: footprint (none) -> Fuse:Fuse_1206_3216Metric
- J1: footprint (none) -> Connector_USB:USB_C_Receptacle_GCT_USB4085
- J2: footprint (none) -> Connector_FFC-FPC:Hirose_FH12-12S-0.5SH_1x12-1MP_P0.50mm_Horizontal
- J3: footprint (none) -> Connector_Coaxial:U.FL_Hirose_U.FL-R-SMT-1_Vertical
- R1, R2, R3, R4, R5, R6: footprint (none) -> Resistor_SMD:R_0603_1608Metric
- SW1: footprint (none) -> Rotary_Encoder:RotaryEncoder_Alps_EC11E-Switch_Vertical_H20mm
- SW3, SW4: footprint (none) -> Button_Switch_SMD:SW_SPST_PTS645Sx43SMTR92
Connections:
- net at U4.4 (I/O2): now also R8.2; no longer U1.13 (USB_D-)
- net at U4.6 (I/O1): now also R7.2; no longer U1.14 (USB_D+)
- new net: R8.1, U1.13 (USB_D-)
- new net: R7.1, U1.14 (USB_D+)
Changed lines of the file:
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@@
 	(wire
 		(pts
-			(xy 57.15 78.74) (xy 57.15 86.36)
+			(xy 66.04 35.56) (xy 66.04 44.45)
 		)
 		(stroke
@@
 	(wire
 		(pts
-			(xy 21.59 87.63) (xy 21.59 90.17)
+			(xy 57.15 78.74) (xy 57.15 86.36)
 		)
 		(stroke
@@
 	(wire
 		(pts
-			(xy 114.3 120.65) (xy 114.3 139.7)
+			(xy 21.59 87.63) (xy 21.59 90.17)
 		)
 		(stroke
@@
 	(wire
 		(pts
-			(xy 44.45 13.97) (xy 44.45 16.51)
+			(xy 114.3 120.65) (xy 114.3 139.7)
 		)
 		(stroke
@@
 	(wire
 		(pts
-			(xy 67.31 12.7) (xy 67.31 46.99)
+			(xy 44.45 13.97) (xy 44.45 16.51)
 		)
 		(stroke
@@
 	(wire
 		(pts
+			(xy 67.31 20.32) (xy 67.31 46.99)
+		)
+		(stroke
+			(width 0)
+			(type default)
+		)
+	)
+	(wire
+		(pts
 			(xy 123.19 82.55) (xy 115.57 82.55)
 		)
@@
 	(wire
 		(pts
-			(xy 66.04 13.97) (xy 66.04 44.45)
-		)
-		(stroke
-			(width 0)
-			(type default)
-		)
-	)
-	(wire
-		(pts
 			(xy 69.85 81.28) (xy 68.58 81.28)
 		)
@@
 	(wire
 		(pts
+			(xy 66.04 13.97) (xy 66.04 27.94)
+		)
+		(stroke
+			(width 0)
+			(type default)
+		)
+	)
+	(wire
+		(pts
 			(xy 163.83 13.97) (xy 163.83 90.17)
 		)
@@
 			)
 		)
-		(property "Footprint" ""
+		(property "Footprint" "Fuse:Fuse_1206_3216Metric"
 			(at 48.26 20.32 0)
 			(hide yes)
@@
 			)
 		)
-		(property "Footprint" ""
+		(property "Footprint" "LED_SMD:LED_0603_1608Metric"
 			(at 86.36 153.67 0)
 			(hide yes)
@@
 			)
 		)
-		(property "Footprint" ""
+		(property "Footprint" "Capacitor_SMD:C_0603_1608Metric"
 			(at 145.7452 64.77 0)
 			(hide yes)
@@
 			)
 		)
-		(property "Footprint" ""
+		(property "Footprint" "Diode_SMD:D_SOD-323"
 			(at 49.53 13.97 0)
 			(hide yes)
@@
 			)
 		)
-		(property "Footprint" ""
+		(property "Footprint" "Capacitor_SMD:C_0603_1608Metric"
 			(at 58.1152 78.74 0)
 			(hide yes)
@@
 			)
 		)
-		(property "Footprint" ""
+		(property "Footprint" "Button_Switch_SMD:SW_SPST_PTS645Sx43SMTR92"
 			(at 121.92 50.8 0)
 			(hide yes)
@@
 			)
 		)
-		(property "Footprint" ""
+		(property "Footprint" "Connector_Coaxial:U.FL_Hirose_U.FL-R-SMT-1_Vertical"
 			(at 93.98 59.69 0)
 			(hide yes)
@@
 			)
 		)
-		(property "Footprint" ""
+		(property "Footprint" "Connector_USB:USB_C_Receptacle_GCT_USB4085"
 			(at 27.94 46.99 0)
 			(hide yes)
@@
 			)
 		)
-		(property "Footprint" ""
+		(property "Footprint" "Resistor_SMD:R_0603_1608Metric"
 			(at 29.972 101.6 90)
 			(hide yes)
@@
 			)
 		)
-		(property "Footprint" ""
+		(property "Footprint" "Button_Switch_SMD:SW_SPST_PTS645Sx43SMTR92"
 			(at 134.62 50.8 0)
 			(hide yes)
@@
 	)
 	(symbol
+		(lib_id "Device:R")
+		(at 67.31 16.51 0)
+		(unit 1)
+		(body_style 1)
+		(exclude_from_sim no)
+		(in_bom yes)
+		(on_board yes)
+		(in_pos_files yes)
+		(dnp no)
+		(fields_autoplaced yes)
+		(property "Reference" "R8"
+			(at 69.85 15.2399 0)
+			(show_name no)
+			(do_not_autoplace no)
+			(effects
+				(font
+					(size 1.27 1.27)
+				)
+				(justify left)
+			)
+		)
+		(property "Value" "22"
+			(at 69.85 17.7799 0)
+			(show_name no)
+			(do_not_autoplace no)
+			(effects
+				(font
+					(size 1.27 1.27)
+				)
+				(justify left)
+			)
+		)
+		(property "Footprint" "Resistor_SMD:R_0603_1608Metric"
+			(at 65.532 16.51 90)
+			(hide yes)
+			(show_name no)
+			(do_not_autoplace no)
+			(effects
+				(font
+					(size 1.27 1.27)
+				)
+			)
+		)
+		(property "Datasheet" ""
+			(at 67.31 16.51 0)
+			(hide yes)
+			(show_name no)
+			(do_not_autoplace no)
+			(effects
+				(font
+					(size 1.27 1.27)
+				)
+			)
+		)
+		(property "Description" "Resistor"
+			(at 67.31 16.51 0)
+			(hide yes)
+			(show_name no)
+			(do_not_autoplace no)
+			(effects
+				(font
+					(size 1.27 1.27)
+				)
+			)
+		)
+		(pin "1"
+		)
+		(pin "2"
+		)
+		(instances
+			(project "Speed-Limit-Display-v2"
+				(path "/021668ec-f5c9-4c85-a0a5-b6e62158b17d"
+					(reference "R8")
+					(unit 1)
+				)
+			)
+		)
+	)
+	(symbol
 		(lib_id "power:GND")
 		(at 143.51 127 0)
@@
 			)
 		)
-		(property "Footprint" ""
+		(property "Footprint" "Rotary_Encoder:RotaryEncoder_Alps_EC11E-Switch_Vertical_H20mm"
 			(at 92.71 114.046 0)
 			(hide yes)
@@
 			)
 		)
-		(property "Footprint" ""
+		(property "Footprint" "Capacitor_SMD:C_0805_2012Metric"
 			(at 54.3052 99.06 0)
 			(hide yes)
@@
 			)
 		)
-		(property "Footprint" ""
+		(property "Footprint" "Capacitor_SMD:C_0805_2012Metric"
 			(at 82.2452 71.12 0)
 			(hide yes)
@@
 			)
 		)
-		(property "Footprint" ""
+		(property "Footprint" "Resistor_SMD:R_0603_1608Metric"
 			(at 118.872 36.83 90)
 			(hide yes)
@@
 			)
 		)
-		(property "Footprint" ""
+		(property "Footprint" "Resistor_SMD:R_0603_1608Metric"
 			(at 92.202 147.32 90)
 			(hide yes)
@@
 			)
 		)
-		(property "Footprint" ""
+		(property "Footprint" "Connector_FFC-FPC:Hirose_FH12-12S-0.5SH_1x12-1MP_P0.50mm_Horizontal"
 			(at 110.49 160.02 0)
 			(hide yes)
@@
 			)
 		)
-		(property "Footprint" ""
+		(property "Footprint" "Capacitor_SMD:C_0603_1608Metric"
 			(at 105.1052 24.13 0)
 			(hide yes)
@@
 			)
 		)
-		(property "Footprint" ""
+		(property "Footprint" "Resistor_SMD:R_0603_1608Metric"
 			(at 115.062 45.72 90)
 			(hide yes)
@@
 			)
 		)
-		(property "Footprint" ""
+		(property "Footprint" "Resistor_SMD:R_0603_1608Metric"
 			(at 38.862 101.6 90)
 			(hide yes)
@@
 			)
 		)
-		(property "Footprint" ""
+		(property "Footprint" "Capacitor_SMD:C_0603_1608Metric"
 			(at 96.2152 88.9 0)
 			(hide yes)
@@
 			)
 		)
-		(property "Footprint" ""
+		(property "Footprint" "Resistor_SMD:R_0603_1608Metric"
 			(at 117.602 67.31 90)
 			(hide yes)
@@
 			)
 		)
-		(property "Footprint" ""
+		(property "Footprint" "Buzzer_Beeper:Buzzer_Murata_PKMCS0909E"
 			(at 95.885 135.89 90)
 			(hide yes)
@@
 					(unit 1)
 				)
+			)
+		)
+	)
+	(symbol
+		(lib_id "Device:R")
+		(at 66.04 31.75 0)
+		(unit 1)
+		(body_style 1)
+		(exclude_from_sim no)
+		(in_bom yes)
+		(on_board yes)
+		(in_pos_files yes)
+		(dnp no)
+		(fields_autoplaced yes)
+		(property "Reference" "R7"
+			(at 68.58 30.4799 0)
+			(show_name no)
+			(do_not_autoplace no)
+			(effects
+				(font
+					(size 1.27 1.27)
+				)
+				(justify left)
+			)
+		)
+		(property "Value" "22"
+			(at 68.58 33.0199 0)
+			(show_name no)
+			(do_not_autoplace no)
+			(effects
+				(font
+					(size 1.27 1.27)
+				)
+				(justify left)
+			)
+		)
+		(property "Footprint" "Resistor_SMD:R_0603_1608Metric"
+			(at 64.262 31.75 90)
+			(hide yes)
+			(show_name no)
+			(do_not_autoplace no)
+			(effects
+				(font
+					(size 1.27 1.27)
+				)
+			)
+		)
+		(property "Datasheet" ""
+			(at 66.04 31.75 0)
+			(hide yes)
+			(show_name no)
+			(do_not_autoplace no)
+			(effects
+				(font
+					(size 1.27 1.27)
+				)
+			)
+		)
+		(property "Description" "Resistor"
+			(at 66.04 31.75 0)
+			(hide yes)
+			(show_name no)
+			(do_not_autoplace no)
+			(effects
+				(font
+					(size 1.27 1.27)
+				)
+			)
+		)
+		(pin "2"
+		)
+		(pin "1"
+		)
+		(instances
+			(project "Speed-Limit-Display-v2"
+				(path "/021668ec-f5c9-4c85-a0a5-b6e62158b17d"
+					(reference "R7")
+					(unit 1)
+				)

Commit message: feat: add J4 breakout header, Gerber/ordering docs, final DRC clean
Added 9-pin breakout header (J4) exposing IO35, IO36, IO45, IO46,
TXD0, RXD0, +3V3, +5V, GND for future sensor expansion. Updated
PCB design docs with step-by-step Gerber generation instructions,
PCBWay/JLCPCB ordering guide, component sourcing, and assembly notes.
Final DRC: 0 errors, 2 cosmetic silkscreen warnings only.

Co-Authored-By: Claude Opus 4.6 (1M context) <noreply@anthropic.com>
Parts:
- added J4: Conn_01x09_Pin, Connector_PinHeader_2.54mm:PinHeader_1x09_P2.54mm_Vertical, symbol Connector:Conn_01x09_Pin
- BZ1: footprint Buzzer_Beeper:Buzzer_Murata_PKMCS0909E -> (none)
- C1, C3, C4, C5: footprint Capacitor_SMD:C_0603_1608Metric -> (none)
- C2, C6: footprint Capacitor_SMD:C_0805_2012Metric -> (none)
- D1: footprint LED_SMD:LED_0603_1608Metric -> (none)
- D2: footprint Diode_SMD:D_SOD-323 -> (none)
- F1: footprint Fuse:Fuse_1206_3216Metric -> (none)
- J1: footprint Connector_USB:USB_C_Receptacle_GCT_USB4085 -> (none)
- J2: footprint Connector_FFC-FPC:Hirose_FH12-12S-0.5SH_1x12-1MP_P0.50mm_Horizontal -> (none)
- J3: footprint Connector_Coaxial:U.FL_Hirose_U.FL-R-SMT-1_Vertical -> (none)
- R1, R2, R3, R4, R5, R6: footprint Resistor_SMD:R_0603_1608Metric -> (none)
- R7, R8: value 22 -> R; footprint Resistor_SMD:R_0603_1608Metric -> (none)
- SW1: footprint Rotary_Encoder:RotaryEncoder_Alps_EC11E-Switch_Vertical_H20mm -> (none)
- SW3, SW4: footprint Button_Switch_SMD:SW_SPST_PTS645Sx43SMTR92 -> (none)
Connections:
- net +3V3: now also J4.1 (Pin_1)
- net +5V: now also J4.2 (Pin_2)
- net GND: now also J4.3 (Pin_3)
- net IO46: now reaches U1.16 (IO46)
- net IO46: now also J4.7 (Pin_7)
- net IO45: now reaches U1.26 (IO45)
- net IO45: now also J4.6 (Pin_6)
- net IO35: now reaches U1.28 (IO35)
- net IO35: now also J4.4 (Pin_4)
- net IO36: now reaches U1.29 (IO36)
- net IO36: now also J4.5 (Pin_5)
- net RXD0: now reaches U1.36 (RXD0)
- net RXD0: now also J4.9 (Pin_9)
- net TXD0: now reaches U1.37 (TXD0)
- net TXD0: now also J4.8 (Pin_8)
- no-connect marks 37 -> 31
